File: schematic-design/KnockLockV2.1.kicad_sch (KiCad schematic)
At the start: 51 parts, among them IC1 ESP32-C3-WROOM-02-N4, IC2 LM2575-3.3WT, J1 2477, J2 UJ2-B-HR-G-TH, J3 TBP04R12-500-03BE, J4 UART, J5 Boot Pins, Q1 IRLML6402TRPBF, Q2 BC547B, SW1 SW_Push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

Commit message: V2.1 adjustments
- added all footprints
- added all components to BOM
Parts:
- removed SW1: SW_Push, symbol Switch:SW_Push
- added S1: 2-1977223-8, 219772238, symbol 2-1977223-8:2-1977223-8
- C10: value 0.1uF - ceramic -> 0.1uF; footprint (none) -> Capacitor_THT:C_Rect_L4.0mm_W2.5mm_P2.50mm
- C11: footprint (none) -> Capacitor_THT:C_Radial_D4.0mm_H7.0mm_P1.50mm
- C3: footprint (none) -> Capacitor_THT:C_Radial_D5.0mm_H11.0mm_P2.00mm
- C4, C5, C6, C8: footprint (none) -> Capacitor_THT:C_Rect_L4.0mm_W2.5mm_P2.50mm
- C7: value 1000uF -> 10uF; footprint (none) -> Capacitor_THT:C_Radial_D5.0mm_H11.0mm_P2.00mm
- D2, D3, D4: footprint (none) -> LED_THT:LED_D3.0mm
- F1, F2: footprint (none) -> Fuse:Fuse_BelFuse_0ZRE0012FF_L8.3mm_W3.8mm
- J5, TP4: footprint (none) -> Connector_PinHeader_2.54mm:PinHeader_1x02_P2.54mm_Vertical
- L1: footprint (none) -> Inductor_THT:L_Radial_D9.5mm_P5.00mm_Fastron_07HVP
- R11, R12, R13: footprint (none) -> SamacSys_Parts:RESAD1590W60L630D240
- TP1, TP2, TP3, TP5: footprint (none) -> TestPoint:TestPoint_Pad_D1.5mm
- TP6: footprint (none) -> Connector_PinSocket_2.54mm:PinSocket_1x01_P2.54mm_Vertical
Connections:
- net GND: now also S1.4 (NO_2)
- net MRESET: now also S1.2 (COM_2)
- no-connect marks 16 -> 18
Other:
- moved on the sheet: C6
