File: KnockLock/KnockLock.kicad_pcb (KiCad board)
At the start: 2 copper layers, 120 x 100 mm, 51 parts, among them IC1 ESP32-C3-WROOM-02-N4, IC2 LM2575-3.3WT, J1 2477, J2 UJ2-B-HR-G-TH, J3 TBP04R12-500-03BE, J4 UART, J5 Boot Pins, Q1 IRLML6402TRPBF, Q2 BC547B, U1 ADXL345BCCZ-RL7

Commit message: Made first draft of pcb design, modified existing library symbol, changes to BOM, changes to schematic
Parts:
- J1: value 2477 -> Screw_Terminal_01x02; footprint SamacSys_Parts:2477 -> TerminalBlock:TerminalBlock_bornier-2_P5.08mm
- J2: value UJ2-B-HR-G-TH -> USB3145-30-1-A; footprint SamacSys_Parts:UJ2BHRGTH -> SamacSys_Parts:USB3145301A
- moved C1 398.5 mm to (23.7, 73.8)
- moved TP1 394.2 mm to (25.0, 97.7), turned to 180 degrees
- moved TP3 389.9 mm to (24.5, 67.3)
- moved TP2 378.5 mm to (40.9, 101.8)
- moved C3 373.0 mm to (43.2, 73.7)
- moved C11 368.6 mm to (46.5, 83.5), turned to 180 degrees
- moved D5 366.5 mm to (31.4, 98.0), turned to 90 degrees
- moved D1 364.6 mm to (31.2, 67.7), turned to 90 degrees
- moved TP4 363.7 mm to (80.6, 96.3)
- moved D6 359.8 mm to (37.5, 98.1), turned to 90 degrees
- moved C9 358.4 mm to (56.8, 61.6)
- moved TP6 348.7 mm to (62.3, 57.4)
- moved TP5 347.4 mm to (66.3, 57.3)
- moved R1 346.8 mm to (61.4, 93.3)
- moved R2 346.5 mm to (61.4, 96.4)
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Connections:
- J2 pad 4: GND -> unconnected-(J2-Pad4)
Other:
- board size 120 x 100 mm -> 90 x 60 mm
- board text added: "Group 04 KnockLock"
