File: pcb-design/KnockLockV1.1.kicad_pcb (KiCad board)
At the start: 2 copper layers, 90 x 60 mm, 51 parts, among them IC1 ESP32-C3-WROOM-02-N4, IC2 LM2575-3.3WT, J1 Screw_Terminal_01x02, J2 USB3145-30-1-A, J3 TBP04R12-500-03BE, J4 UART, J5 Boot Pins, Q1 IRLML6402TRPBF, Q2 BC547B

Commit message: Minor adjustments to PCB design, fixed DRCs
Parts:
- moved C3 4.40 mm to (45.1, 73.7)
Routing:
- net +3.3V: track 16.9 -> 0.00 mm
Changed lines of the file:
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@@
 			(outputformat 1)
 			(mirror no)
-			(drillshape 0)
+			(drillshape 1)
 			(scaleselection 1)
-			(outputdirectory "../pcb-design/")
+			(outputdirectory "")
 		)
 	)
@@
 		(tags "C Rect series Radial pin pitch 2.50mm length 4mm width 2.5mm Capacitor")
 		(property "Reference" "C4"
-			(at 1.25 -2.5052 0)
+			(at 1.426162 2.634822 0)
 			(layer "F.SilkS")
 			(effects
@@
 		)
 		(property "Value" "0.1uF"
-			(at -2.0438 -1.5752 180)
+			(at 0.026162 3.714822 180)
 			(layer "F.Fab")
 			(effects
@@
 	(footprint "Capacitor_THT:C_Radial_D5.0mm_H11.0mm_P2.00mm"
 		(layer "F.Cu")
-		(at 49.47 74.19 180)
+		(at 45.1 73.68 180)
 		(descr "C, Radial series, Radial, pin pitch=2.00mm, diameter=5mm, height=11mm, Non-Polar Electrolytic Capacitor")
 		(tags "C Radial series Radial pin pitch 2.00mm diameter 5mm height 11mm Non-Polar Electrolytic Capacitor")
@@
 		)
 		(property "Value" "10uF"
-			(at 5.25 -1.98 0)
+			(at -2.18 3.52 0)
 			(layer "F.Fab")
 			(effects
@@
 		)
 	)
-	(segment
-		(start 55.4338 76.0738)
-		(end 54.2748 76.0738)
-		(width 0.7)
-		(layer "F.Cu")
-		(net 5)
-	)
-	(segment
-		(start 58.8309 78.1893)
-		(end 57.5493 78.1893)
-		(width 0.7)
-		(layer "F.Cu")
-		(net 5)
-	)
-	(segment
-		(start 54.2748 76.0738)
-		(end 49.3538 76.0738)
-		(width 0.7)
-		(layer "F.Cu")
-		(net 5)
-	)
-	(segment
-		(start 57.5493 78.1893)
-		(end 55.4338 76.0738)
-		(width 0.7)
-		(layer "F.Cu")
-		(net 5)
-	)
-	(segment
-		(start 49.3538 76.0738)
-		(end 47.47 74.19)
-		(width 0.7)
-		(layer "F.Cu")
-		(net 5)
-	)
-	(segment
-		(start 63.37 61.99)
-		(end 62.3 63.06)
-		(width 0.7)
-		(layer "F.Cu")
-		(net 5)
-	)
-	(segment
-		(start 65.74 61.99)
-		(end 63.37 61.99)
-		(width 0.7)
-		(layer "F.Cu")
-		(net 5)
-	)
 	(zone
